File: sheesh.kicad_pcb (KiCad board)
At the start: 2 copper layers, 234.7 x 104.6 mm, 104 parts, among them J1 3305-0-15-80-47-27-10-0, J10 3305-0-15-80-47-27-10-0, J11 3305-0-15-80-47-27-10-0, J12 3305-0-15-80-47-27-10-0, J13 3305-0-15-80-47-27-10-0, J14 3305-0-15-80-47-27-10-0, J15 3305-0-15-80-47-27-10-0, J16 3305-0-15-80-47-27-10-0, J17 3305-0-15-80-47-27-10-0, J18 3305-0-15-80-47-27-10-0, J19 3305-0-15-80-47-27-10-0, J2 3305-0-15-80-47-27-10-0, J20 3305-0-15-80-47-27-10-0, J21 3305-0-15-80-47-27-10-0, J22 3305-0-15-80-47-27-10-0, J23 3305-0-15-80-47-27-10-0, J24 3305-0-15-80-47-27-10-0, J25 3305-0-15-80-47-27-10-0, J26 3305-0-15-80-47-27-10-0, J27 3305-0-15-80-47-27-10-0, J28 3305-0-15-80-47-27-10-0, J29 3305-0-15-80-47-27-10-0, J3 3305-0-15-80-47-27-10-0, J30 3305-0-15-80-47-27-10-0, J31 3305-0-15-80-47-27-10-0, J32 3305-0-15-80-47-27-10-0, J33 3305-0-15-80-47-27-10-0, J34 3305-0-15-80-47-27-10-0, J35 3305-0-15-80-47-27-10-0, J36 3305-0-15-80-47-27-10-0, J37 3305-0-15-80-47-27-10-0, J38 3305-0-15-80-47-27-10-0, J39 3305-0-15-80-47-27-10-0, J4 3305-0-15-80-47-27-10-0, J40 3305-0-15-80-47-27-10-0, J41 3305-0-15-80-47-27-10-0, J42 3305-0-15-80-47-27-10-0, J43 3305-0-15-80-47-27-10-0, J44 3305-0-15-80-47-27-10-0, J45 3305-0-15-80-47-27-10-0, J46 3305-0-15-80-47-27-10-0, J47 3305-0-15-80-47-27-10-0, J48 3305-0-15-80-47-27-10-0, J49 3305-0-15-80-47-27-10-0, J5 3305-0-15-80-47-27-10-0, J50 3305-0-15-80-47-27-10-0, J51 3305-0-15-80-47-27-10-0, J52 3305-0-15-80-47-27-10-0, J53 3305-0-15-80-47-27-10-0, J54 3305-0-15-80-47-27-10-0, J55 3305-0-15-80-47-27-10-0, J56 3305-0-15-80-47-27-10-0, J57 310-13-107-41-001000, J58 310-13-107-41-001000, J59 YZ00615050R-04, J6 3305-0-15-80-47-27-10-0, J60 YZ00615050R-04, J61 YZ00615050R-04, J62 YZ00615050R-04, J63 YZ00615050R-04, J64 310-13-107-41-001000, J65 310-13-107-41-001000, J66 YZ00615050R-04, J67 YZ00615050R-04, J68 YZ00615050R-04, J69 YZ00615050R-04, J7 3305-0-15-80-47-27-10-0, J70 YZ00615050R-04, J8 3305-0-15-80-47-27-10-0, J9 3305-0-15-80-47-27-10-0, SW1 SW_Push, SW10 SW_Push, SW11 SW_Push, SW12 SW_Push, SW13 SW_Push, SW14 SW_Push, SW15 SW_Push, SW16 SW_Push, SW17 SW_Push, SW18 SW_Push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

Commit message: switch to diodes
Parts:
- removed J59, J60, J62, J63, J66, J67, J69, J70: YZ00615050R-04, Sheesh:YZ00615050R-04
- added ?: , , F.Cu at (158.2, 111.0)
- added ?: , , F.Cu at (161.8, 92.5)
- added ?: , , F.Cu at (158.2, 112.3)
- added ?: , , F.Cu at (161.9, 73.9)
- added ?: , , F.Cu at (161.9, 113.6)
- added ?: , , F.Cu at (158.1, 75.2)
- added ?: , , F.Cu at (158.0, 91.2)
- added ?: , , F.Cu at (161.8, 93.8)
- added ?: , , F.Cu at (161.7, 91.3)
- added ?: , , F.Cu at (161.9, 112.3)
- added ?: , , F.Cu at (158.0, 72.7)
- added ?: , , F.Cu at (158.1, 92.4)
- added ?: , , F.Cu at (158.2, 113.5)
- added ?: , , F.Cu at (158.1, 93.6)
- added ?: , , F.Cu at (161.9, 75.2)
- added ?: , , F.Cu at (158.1, 73.9)
- added ?: , , F.Cu at (161.8, 72.7)
- added ?: , , F.Cu at (161.8, 111.1)
- added D1: CDSQC4148-HF, Sheesh:X1-DFN1006-2_L1.0-W0.6-RD, F.Cu at (171.9, 106.3)
- added D10: CDSQC4148-HF, Sheesh:X1-DFN1006-2_L1.0-W0.6-RD, F.Cu at (188.0, 96.0)
- added D11: CDSQC4148-HF, Sheesh:X1-DFN1006-2_L1.0-W0.6-RD, F.Cu at (208.3, 92.5)
- added D12: CDSQC4148-HF, Sheesh:X1-DFN1006-2_L1.0-W0.6-RD, F.Cu at (224.7, 100.8)
- added D13: CDSQC4148-HF, Sheesh:X1-DFN1006-2_L1.0-W0.6-RD, F.Cu at (168.9, 106.3)
- added D14: CDSQC4148-HF, Sheesh:X1-DFN1006-2_L1.0-W0.6-RD, F.Cu at (189.0, 96.1)
- added D15: CDSQC4148-HF, Sheesh:X1-DFN1006-2_L1.0-W0.6-RD, F.Cu at (93.1, 101.2)
- added D16: CDSQC4148-HF, Sheesh:X1-DFN1006-2_L1.0-W0.6-RD, F.Cu at (109.7, 93.0)
- added D17: CDSQC4148-HF, Sheesh:X1-DFN1006-2_L1.0-W0.6-RD, F.Cu at (128.9, 96.4)
- added D18: CDSQC4148-HF, Sheesh:X1-DFN1006-2_L1.0-W0.6-RD, F.Cu at (147.8, 106.2)
- added D19: CDSQC4148-HF, Sheesh:X1-DFN1006-2_L1.0-W0.6-RD, F.Cu at (94.1, 101.0)
- added D2: CDSQC4148-HF, Sheesh:X1-DFN1006-2_L1.0-W0.6-RD, F.Cu at (191.0, 96.2)
- added D20: CDSQC4148-HF, Sheesh:X1-DFN1006-2_L1.0-W0.6-RD, F.Cu at (110.7, 92.8)
- added D21: CDSQC4148-HF, Sheesh:X1-DFN1006-2_L1.0-W0.6-RD, F.Cu at (129.9, 96.3)
- added D22: CDSQC4148-HF, Sheesh:X1-DFN1006-2_L1.0-W0.6-RD, F.Cu at (148.9, 106.2)
- added D23: CDSQC4148-HF, Sheesh:X1-DFN1006-2_L1.0-W0.6-RD, F.Cu at (95.1, 100.8)
- added D24: CDSQC4148-HF, Sheesh:X1-DFN1006-2_L1.0-W0.6-RD, F.Cu at (111.7, 92.6)
- added D25: CDSQC4148-HF, Sheesh:X1-DFN1006-2_L1.0-W0.6-RD, F.Cu at (131.9, 96.1)
- added D26: CDSQC4148-HF, Sheesh:X1-DFN1006-2_L1.0-W0.6-RD, F.Cu at (149.9, 106.2)
- added D27: CDSQC4148-HF, Sheesh:X1-DFN1006-2_L1.0-W0.6-RD, F.Cu at (130.9, 96.2)
- added D28: CDSQC4148-HF, Sheesh:X1-DFN1006-2_L1.0-W0.6-RD, F.Cu at (150.9, 106.2)
- added D3: CDSQC4148-HF, Sheesh:X1-DFN1006-2_L1.0-W0.6-RD, F.Cu at (210.3, 92.8)
- added D4: CDSQC4148-HF, Sheesh:X1-DFN1006-2_L1.0-W0.6-RD, F.Cu at (226.7, 101.1)
- added D5: CDSQC4148-HF, Sheesh:X1-DFN1006-2_L1.0-W0.6-RD, F.Cu at (170.9, 106.3)
- added D6: CDSQC4148-HF, Sheesh:X1-DFN1006-2_L1.0-W0.6-RD, F.Cu at (190.0, 96.1)
- added D7: CDSQC4148-HF, Sheesh:X1-DFN1006-2_L1.0-W0.6-RD, F.Cu at (209.3, 92.7)
- added D8: CDSQC4148-HF, Sheesh:X1-DFN1006-2_L1.0-W0.6-RD, F.Cu at (225.7, 100.9)
- added D9: CDSQC4148-HF, Sheesh:X1-DFN1006-2_L1.0-W0.6-RD, F.Cu at (169.9, 106.3)
- J57, J58, J64, J65: value 310-13-107-41-001000 -> MF254V-11-07-0743
- moved SW30 1.36 mm to (69.2, 89.7)
- moved U3 1.19 mm to (228.6, 59.3), turned to 35 degrees
- moved SW29 0.92 mm to (250.4, 89.8)
- moved J20 0.89 mm to (188.7, 106.7)
- moved U1 0.89 mm to (248.9, 99.7)
- moved J64 0.89 mm to (63.5, 101.1)
- moved J52 0.89 mm to (149.4, 116.9)
- moved J6 0.89 mm to (213.2, 69.5)
- moved J11 0.89 mm to (185.3, 87.3)
- moved J43 0.89 mm to (144.4, 97.8)
- moved J8 0.89 mm to (230.0, 78.1)
- moved SW8 0.89 mm to (228.0, 88.9)
- moved J4 0.89 mm to (191.6, 72.9)
- moved J10 0.89 mm to (170.5, 99.8)
- moved SW5 0.89 mm to (170.5, 93.9)
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Connections:
- J1 pad 1: GND -> /row1
- J10 pad 1: /sw5 -> Net-(D5-K)
- J11 pad 1: GND -> /row2
- J12 pad 1: /sw6 -> Net-(D6-K)
- J13 pad 1: GND -> /row2
- J14 pad 1: /sw7 -> Net-(D7-K)
- J15 pad 1: GND -> /row2
- J16 pad 1: /sw8 -> Net-(D8-K)
- J17 pad 1: GND -> /row3
- J18 pad 1: /sw9 -> Net-(D9-K)
- J19 pad 1: GND -> /row3
- J2 pad 1: /sw1 -> Net-(D1-K)
- J20 pad 1: /sw10 -> Net-(D10-K)
- J21 pad 1: GND -> /row3
- J22 pad 1: /sw11 -> Net-(D11-K)
- J23 pad 1: GND -> /row3
- J24 pad 1: /sw12 -> Net-(D12-K)
- J25 pad 1: GND -> /row4
- J26 pad 1: /sw13 -> Net-(D13-K)
- J27 pad 1: GND -> /row4
- J28 pad 1: /sw14 -> Net-(D14-K)
- J29 pad 1: GND -> /row5
- J3 pad 1: GND -> /row1
- J30 pad 1: /sw15 -> Net-(D15-K)
- J31 pad 1: GND -> /row5
- J32 pad 1: /sw16 -> Net-(D16-K)
- J33 pad 1: GND -> /row5
- J34 pad 1: /sw17 -> Net-(D17-K)
- J35 pad 1: GND -> /row5
- J36 pad 1: /sw18 -> Net-(D18-K)
- J37 pad 1: GND -> /row6
- J38 pad 1: /sw19 -> Net-(D19-K)
- J39 pad 1: GND -> /row6
- J4 pad 1: /sw2 -> Net-(D2-K)
- J40 pad 1: /sw20 -> Net-(D20-K)
- J41 pad 1: GND -> /row6
- J42 pad 1: /sw21 -> Net-(D21-K)
- J43 pad 1: GND -> /row6
- J44 pad 1: /sw22 -> Net-(D22-K)
- J45 pad 1: GND -> /row7
- J46 pad 1: /sw23 -> Net-(D23-K)
- J47 pad 1: GND -> /row7
- J48 pad 1: /sw24 -> Net-(D24-K)
- J49 pad 1: GND -> /row7
- J5 pad 1: GND -> /row1
- J50 pad 1: /sw25 -> Net-(D25-K)
- J51 pad 1: GND -> /row7
- J52 pad 1: /sw26 -> Net-(D26-K)
- J53 pad 1: GND -> /row8
- J54 pad 1: /sw27 -> Net-(D27-K)
- J55 pad 1: GND -> /row8
- J56 pad 1: /sw28 -> Net-(D28-K)
- J57 pad 1: /sw3 -> Net-(J57-Pin_1)
- J57 pad 2: /sw2 -> Net-(J57-Pin_2)
- J57 pad 3: /sw1 -> Net-(J57-Pin_3)
- J57 pad 4: /sw7 -> /col4
- J57 pad 5: /sw5 -> /col3
- J57 pad 6: /sw10 -> /col2
- J57 pad 7: /sw11 -> /col1
- J58 pad 4: /sw8 -> /row1
- J58 pad 5: /sw6 -> /row2
- J58 pad 6: /sw9 -> /row3
- J58 pad 7: /sw12 -> /row4
- J6 pad 1: /sw3 -> Net-(D3-K)
- J64 pad 1: /sw27 -> Net-(J64-Pin_1)
- J64 pad 2: /sw28 -> Net-(J64-Pin_2)
- J64 pad 3: /sw23 -> Net-(J64-Pin_3)
- J64 pad 4: /sw17 -> /row5
- J64 pad 5: /sw19 -> /row6
- J64 pad 6: /sw21 -> /row7
- J64 pad 7: /sw24 -> /row8
- J65 pad 4: /sw16 -> /col5
- J65 pad 5: /sw18 -> /col6
- J65 pad 6: /sw20 -> /col7
- J65 pad 7: /sw22 -> /col8
- J7 pad 1: GND -> /row1
- J8 pad 1: /sw4 -> Net-(D4-K)
- J9 pad 1: GND -> /row2
- SW1 pad 1: GND -> /row1
- SW1 pad 2: /sw1 -> Net-(D1-K)
- SW10 pad 1: GND -> /row3
- SW10 pad 2: /sw10 -> Net-(D10-K)
- SW11 pad 1: GND -> /row3
- SW11 pad 2: /sw11 -> Net-(D11-K)
- SW12 pad 1: GND -> /row3
- SW12 pad 2: /sw12 -> Net-(D12-K)
- SW13 pad 1: GND -> /row4
- SW13 pad 2: /sw13 -> Net-(D13-K)
- SW14 pad 1: GND -> /row4
- SW14 pad 2: /sw14 -> Net-(D14-K)
- SW15 pad 1: GND -> /row5
- SW15 pad 2: /sw15 -> Net-(D15-K)
- SW16 pad 1: GND -> /row5
- SW16 pad 2: /sw16 -> Net-(D16-K)
- SW17 pad 1: GND -> /row5
- SW17 pad 2: /sw17 -> Net-(D17-K)
- SW18 pad 1: GND -> /row5
- SW18 pad 2: /sw18 -> Net-(D18-K)
- SW19 pad 1: GND -> /row6
- SW19 pad 2: /sw19 -> Net-(D19-K)
- SW2 pad 1: GND -> /row1
- SW2 pad 2: /sw2 -> Net-(D2-K)
- SW20 pad 1: GND -> /row6
- SW20 pad 2: /sw20 -> Net-(D20-K)
- SW21 pad 1: GND -> /row6
- SW21 pad 2: /sw21 -> Net-(D21-K)
- SW22 pad 1: GND -> /row6
- SW22 pad 2: /sw22 -> Net-(D22-K)
- SW23 pad 1: GND -> /row7
- SW23 pad 2: /sw23 -> Net-(D23-K)
- SW24 pad 1: GND -> /row7
- SW24 pad 2: /sw24 -> Net-(D24-K)
- SW25 pad 1: GND -> /row7
- SW25 pad 2: /sw25 -> Net-(D25-K)
- SW26 pad 1: GND -> /row7
- SW26 pad 2: /sw26 -> Net-(D26-K)
- SW27 pad 1: GND -> /row8
- SW27 pad 2: /sw27 -> Net-(D27-K)
- SW28 pad 1: GND -> /row8
- SW28 pad 2: /sw28 -> Net-(D28-K)
- SW3 pad 1: GND -> /row1
- SW3 pad 2: /sw3 -> Net-(D3-K)
- SW4 pad 1: GND -> /row1
- SW4 pad 2: /sw4 -> Net-(D4-K)
- SW5 pad 1: GND -> /row2
- SW5 pad 2: /sw5 -> Net-(D5-K)
- SW6 pad 1: GND -> /row2
- SW6 pad 2: /sw6 -> Net-(D6-K)
- SW7 pad 1: GND -> /row2
- SW7 pad 2: /sw7 -> Net-(D7-K)
- SW8 pad 1: GND -> /row2
- SW8 pad 2: /sw8 -> Net-(D8-K)
- SW9 pad 1: GND -> /row3
- SW9 pad 2: /sw9 -> Net-(D9-K)
- U1 pad 1: /sw3 -> Net-(J57-Pin_1)
- U1 pad 10: /sw6 -> /row2
- U1 pad 11: /sw8 -> /row1
- U1 pad 2: /sw2 -> Net-(J57-Pin_2)
- U1 pad 3: /sw1 -> Net-(J57-Pin_3)
- U1 pad 4: /sw7 -> /col4
- U1 pad 5: /sw5 -> /col3
- U1 pad 6: /sw10 -> /col2
- U1 pad 7: /sw11 -> /col1
- U1 pad 8: /sw12 -> /row4
- U1 pad 9: /sw9 -> /row3
- U2 pad 1: /sw27 -> Net-(J64-Pin_1)
- U2 pad 10: /sw18 -> /col6
- U2 pad 11: /sw16 -> /col5
- U2 pad 2: /sw28 -> Net-(J64-Pin_2)
- U2 pad 3: /sw23 -> Net-(J64-Pin_3)
- U2 pad 4: /sw17 -> /row5
- U2 pad 5: /sw19 -> /row6
- U2 pad 6: /sw21 -> /row7
- U2 pad 7: /sw24 -> /row8
- U2 pad 8: /sw22 -> /col8
- U2 pad 9: /sw20 -> /col7
Routing:
- net Net-(D27-K): track 0.00 -> 150.3 mm
- net Net-(D14-K): track 0.00 -> 148.1 mm
- net /row1: track 0.00 -> 113.4 mm
- net /row2: track 0.00 -> 111.5 mm
- net /row5: track 0.00 -> 105.2 mm
- net /row3: track 0.00 -> 101.8 mm
- net /row6: track 0.00 -> 98.3 mm
- net /sw9: track 93.4 -> 0.00 mm
- net /row7: track 0.00 -> 92.1 mm
- net /sw26: track 87.2 -> 0.00 mm, vias 1 -> 0
- net /sw18: track 82.6 -> 0.00 mm
- net /col1: track 0.00 -> 82.1 mm
- net /sw17: track 80.4 -> 0.00 mm
- net /col8: track 0.00 -> 78.8 mm
- net /sw1: track 78.7 -> 0.00 mm
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Other:
- outline, holes or cut-outs redrawn
