File: sheesh.kicad_sch (KiCad schematic)
At the start: 124 parts, among them J1 3305-0-15-80-47-27-10-0, J10 3305-0-15-80-47-27-10-0, J11 3305-0-15-80-47-27-10-0, J12 3305-0-15-80-47-27-10-0, J13 3305-0-15-80-47-27-10-0, J14 3305-0-15-80-47-27-10-0, J15 3305-0-15-80-47-27-10-0, J16 3305-0-15-80-47-27-10-0, J17 3305-0-15-80-47-27-10-0, J18 3305-0-15-80-47-27-10-0, J19 3305-0-15-80-47-27-10-0, J2 3305-0-15-80-47-27-10-0, J20 3305-0-15-80-47-27-10-0, J21 3305-0-15-80-47-27-10-0, J22 3305-0-15-80-47-27-10-0, J23 3305-0-15-80-47-27-10-0, J24 3305-0-15-80-47-27-10-0, J25 3305-0-15-80-47-27-10-0, J26 3305-0-15-80-47-27-10-0, J27 3305-0-15-80-47-27-10-0, J28 3305-0-15-80-47-27-10-0, J29 3305-0-15-80-47-27-10-0, J3 3305-0-15-80-47-27-10-0, J30 3305-0-15-80-47-27-10-0, J31 3305-0-15-80-47-27-10-0, J32 3305-0-15-80-47-27-10-0, J33 3305-0-15-80-47-27-10-0, J34 3305-0-15-80-47-27-10-0, J35 3305-0-15-80-47-27-10-0, J36 3305-0-15-80-47-27-10-0, J37 3305-0-15-80-47-27-10-0, J38 3305-0-15-80-47-27-10-0, J39 3305-0-15-80-47-27-10-0, J4 3305-0-15-80-47-27-10-0, J40 3305-0-15-80-47-27-10-0, J41 3305-0-15-80-47-27-10-0, J42 3305-0-15-80-47-27-10-0, J43 3305-0-15-80-47-27-10-0, J44 3305-0-15-80-47-27-10-0, J45 3305-0-15-80-47-27-10-0, J46 3305-0-15-80-47-27-10-0, J47 3305-0-15-80-47-27-10-0, J48 3305-0-15-80-47-27-10-0, J49 3305-0-15-80-47-27-10-0, J5 3305-0-15-80-47-27-10-0, J50 3305-0-15-80-47-27-10-0, J51 3305-0-15-80-47-27-10-0, J52 3305-0-15-80-47-27-10-0, J53 3305-0-15-80-47-27-10-0, J54 3305-0-15-80-47-27-10-0, J55 3305-0-15-80-47-27-10-0, J56 3305-0-15-80-47-27-10-0, J57 MF254V-11-07-0743, J58 MF254V-11-07-0743, J6 3305-0-15-80-47-27-10-0, J61 YZ00615050R-04, J64 MF254V-11-07-0743, J65 MF254V-11-07-0743, J68 YZ00615050R-04, J7 3305-0-15-80-47-27-10-0, J8 3305-0-15-80-47-27-10-0, J9 3305-0-15-80-47-27-10-0, SW1 SW_Push, SW10 SW_Push, SW11 SW_Push, SW12 SW_Push, SW13 SW_Push, SW14 SW_Push, SW15 SW_Push, SW16 SW_Push, SW17 SW_Push, SW18 SW_Push, SW19 SW_Push, SW2 SW_Push, SW20 SW_Push, SW21 SW_Push, SW22 SW_Push, SW23 SW_Push, SW24 SW_Push, SW25 SW_Push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

Commit message: correct diode text and part number
Parts:
- D1, D10, D11, D12, D13, D14, D15, D16, D17, D18, D19, D2, D20, D21, D22, D23, D24, D25, D26, D27, D28, D3, D4, D5, D6, D7, D8, D9: LCSC (none) -> C6341459; LCSC Part C6341459 -> (none)
- U3, U4: LCSC Part C2902345 -> (none)
Changed lines of the file:
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@@
 			)
 		)
-		(property "LCSC Part" "C2902345"
-			(at 132.08 163.83 0)
-			(effects
-				(font
-					(size 1.27 1.27)
-				)
-				(hide yes)
-			)
-		)
 		(property "Sim.Device" ""
 			(at 132.08 176.53 0)
@@
 			)
 		)
-		(property "LCSC Part" "C6341459"
-			(at 82.55 73.66 0)
+		(property "LCSC" "C6341459"
+			(at 82.55 63.5 0)
 			(effects
 				(font
@@
 			)
 		)
-		(property "LCSC Part" "C6341459"
-			(at 49.53 96.52 0)
+		(property "LCSC" "C6341459"
+			(at 49.53 86.36 0)
 			(effects
 				(font
@@
 			)
 		)
-		(property "LCSC Part" "C2902345"
-			(at 69.85 163.83 0)
-			(effects
-				(font
-					(size 1.27 1.27)
-				)
-				(hide yes)
-			)
-		)
 		(property "Sim.Device" ""
 			(at 69.85 176.53 0)
@@
 			)
 		)
-		(property "LCSC Part" "C6341459"
-			(at 118.11 63.5 0)
+		(property "LCSC" "C6341459"
+			(at 118.11 53.34 0)
 			(effects
 				(font
@@
 			)
 		)
-		(property "LCSC Part" "C6341459"
-			(at 153.67 146.05 0)
+		(property "LCSC" "C6341459"
+			(at 153.67 135.89 0)
 			(effects
 				(font
@@
 			)
 		)
-		(property "LCSC Part" "C6341459"
-			(at 82.55 96.52 0)
+		(property "LCSC" "C6341459"
+			(at 82.55 86.36 0)
 			(effects
 				(font
@@
 			)
 		)
-		(property "LCSC Part" "C6341459"
-			(at 118.11 146.05 0)
+		(property "LCSC" "C6341459"
+			(at 118.11 135.89 0)
 			(effects
 				(font
@@
 			)
 		)
-		(property "LCSC Part" "C6341459"
-			(at 153.67 73.66 0)
+		(property "LCSC" "C6341459"
+			(at 153.67 63.5 0)
 			(effects
 				(font
@@
 			)
 		)
-		(property "LCSC Part" "C6341459"
-			(at 153.67 113.03 0)
+		(property "LCSC" "C6341459"
+			(at 153.67 102.87 0)
 			(effects
 				(font
@@
 			)
 		)
-		(property "LCSC Part" "C6341459"
-			(at 49.53 123.19 0)
+		(property "LCSC" "C6341459"
+			(at 49.53 113.03 0)
 			(effects
 				(font
@@
 			)
 		)
-		(property "LCSC Part" "C6341459"
-			(at 118.11 83.82 0)
+		(property "LCSC" "C6341459"
+			(at 118.11 73.66 0)
 			(effects
 				(font
@@
 			)
 		)
-		(property "LCSC Part" "C6341459"
-			(at 118.11 73.66 0)
+		(property "LCSC" "C6341459"
+			(at 118.11 63.5 0)
 			(effects
 				(font
@@
 			)
 		)
-		(property "LCSC Part" "C6341459"
-			(at 82.55 113.03 0)
+		(property "LCSC" "C6341459"
+			(at 82.55 102.87 0)
 			(effects
 				(font
@@
 			)
 		)
-		(property "LCSC Part" "C6341459"
-			(at 49.53 83.82 0)
+		(property "LCSC" "C6341459"
+			(at 49.53 73.66 0)
 			(effects
 				(font
@@
 			)
 		)
-		(property "LCSC Part" "C6341459"
-			(at 82.55 123.19 0)
+		(property "LCSC" "C6341459"
+			(at 82.55 113.03 0)
 			(effects
 				(font
@@
 			)
 		)
-		(property "LCSC Part" "C6341459"
-			(at 153.67 133.35 0)
+		(property "LCSC" "C6341459"
+			(at 153.67 123.19 0)
 			(effects
 				(font
@@
 			)
 		)
-		(property "LCSC Part" "C6341459"
-			(at 153.67 63.5 0)
+		(property "LCSC" "C6341459"
+			(at 153.67 53.34 0)
 			(effects
 				(font
@@
 			)
 		)
-		(property "LCSC Part" "C6341459"
-			(at 49.53 113.03 0)
+		(property "LCSC" "C6341459"
+			(at 49.53 102.87 0)
 			(effects
 				(font
@@
 			)
 		)
-		(property "LCSC Part" "C6341459"
-			(at 82.55 83.82 0)
+		(property "LCSC" "C6341459"
+			(at 82.55 73.66 0)
 			(effects
 				(font
@@
 			)
 		)
-		(property "LCSC Part" "C6341459"
-			(at 82.55 133.35 0)
+		(property "LCSC" "C6341459"
+			(at 82.55 123.19 0)
 			(effects
 				(font
@@
 			)
 		)
-		(property "LCSC Part" "C6341459"
-			(at 49.53 73.66 0)
+		(property "LCSC" "C6341459"
+			(at 49.53 63.5 0)
 			(effects
 				(font
@@
 			)
 		)
-		(property "LCSC Part" "C6341459"
-			(at 153.67 123.19 0)
+		(property "LCSC" "C6341459"
+			(at 153.67 113.03 0)
 			(effects
 				(font
@@
 			)
 		)
-		(property "LCSC Part" "C6341459"
-			(at 118.11 133.35 0)
+		(property "LCSC" "C6341459"
+			(at 118.11 123.19 0)
 			(effects
 				(font
@@
 			)
 		)
-		(property "LCSC Part" "C6341459"
-			(at 118.11 113.03 0)
+		(property "LCSC" "C6341459"
+			(at 118.11 102.87 0)
 			(effects
 				(font
@@
 			)
 		)
-		(property "LCSC Part" "C6341459"
-			(at 82.55 63.5 0)
+		(property "LCSC" "C6341459"
+			(at 82.55 53.34 0)
 			(effects
 				(font
@@
 			)
 		)
-		(property "LCSC Part" "C6341459"
-			(at 118.11 123.19 0)
+		(property "LCSC" "C6341459"
+			(at 118.11 113.03 0)
 			(effects
 				(font
@@
 			)
 		)
-		(property "LCSC Part" "C6341459"
-			(at 49.53 133.35 0)
+		(property "LCSC" "C6341459"
+			(at 49.53 123.19 0)
 			(effects
 				(font
@@
 			)
 		)
-		(property "LCSC Part" "C6341459"
-			(at 153.67 83.82 0)
+		(property "LCSC" "C6341459"
+			(at 153.67 73.66 0)
 			(effects
 				(font
@@
 			)
 		)
-		(property "LCSC Part" "C6341459"
-			(at 49.53 63.5 0)
+		(property "LCSC" "C6341459"
+			(at 49.53 53.34 0)
 			(effects
 				(font
